Commit message: feat: model upload on gzb

File: myagv_description/urdf/myagv_gazebo.urdf.xacro (robot description, xacro)
@@ -4,16 +4,17 @@
   <xacro:arg name="ros2_control_config" default=""/>
   <!-- Dimensions (approximate, tune with measured data when available) -->
-  <xacro:property name="base_length" value="0.43"/>
-  <xacro:property name="base_width" value="0.33"/>
-  <xacro:property name="base_height" value="0.12"/>
-  <xacro:property name="base_mass" value="14.0"/>
-  <xacro:property name="wheel_radius" value="0.05"/>
-  <xacro:property name="wheel_width" value="0.045"/>
+  <xacro:property name="base_length" value="0.31115"/>
+  <xacro:property name="base_width" value="0.23"/>
+  <xacro:property name="base_height" value="0.11"/>
+  <xacro:property name="base_mass" value="4.16"/>
+  <xacro:property name="wheel_radius" value="0.04"/>
+  <xacro:property name="wheel_width" value="0.032"/>
   <xacro:property name="wheel_mass" value="0.8"/>
-  <xacro:property name="wheel_offset_x" value="0.18"/>
-  <xacro:property name="wheel_offset_y" value="0.17"/>
+  <xacro:property name="wheel_offset_x" value="0.10555"/>
+  <xacro:property name="wheel_offset_y" value="0.10525"/>
   <xacro:property name="imu_height" value="${wheel_radius + base_height + 0.05}"/>
   <xacro:property name="lidar_height" value="${wheel_radius + base_height + 0.08}"/>
   <xacro:property name="camera_height" value="${wheel_radius + base_height + 0.15}"/>
+  <xacro:property name="mesh_path" value="$(find myagv_description)/meshes"/>
   <xacro:property name="ros2_control_config_path" value="$(arg ros2_control_config)"/>
   <!-- Helper macros -->
@@ -49,5 +50,7 @@
     <parent link="base_footprint"/>
     <child link="base_link"/>
+    <!-- <origin xyz="0 0.0045 0" rpy="0 0 0"/> -->
     <origin xyz="0 0 0" rpy="0 0 0"/>
+    <axis xyz="0 0 1"/>
   </joint>
   <!-- Base link with visuals and collision -->
@@ -59,19 +62,43 @@
                         origin_xyz="0 0 ${wheel_radius + base_height/2.0}"/>
     <visual>
-      <origin xyz="0 0 0" rpy="0 0 0"/>
-      <geometry>
-        <mesh filename="package://myagv_description/meshes/myagv_base.dae" scale="1 1 1"/>
-      </geometry>
-    </visual>
-    <visual>
-      <origin xyz="0 0 0" rpy="0 0 0"/>
-      <geometry>
-        <mesh filename="package://myagv_description/meshes/myagv_up.dae" scale="1 1 1"/>
-      </geometry>
-    </visual>
-    <collision>
-      <origin xyz="0 0 ${wheel_radius + base_height/2.0}" rpy="0 0 0"/>
-      <geometry>
-        <box size="${base_length} ${base_width} ${base_height}"/>
+      <origin xyz="-0.0055 0.0045 0" rpy="0 0 0"/>
+      <geometry>
+        <mesh filename="file://${mesh_path}/myagv_base.dae" scale="1 1 1"/>
+      </geometry>
+      <material name="black">
+          <color rgba="0.7 0.7 0.0 1.0"/>
+      </material>
+    </visual>
+    <visual>
+      <origin xyz="-0.0055 0.0045 0" rpy="0 0 0"/>
+      <geometry>
+        <mesh filename="file://${mesh_path}/myagv_up.dae" scale="1 1 1"/>
+      </geometry>
+      <material name="black">
+          <color rgba="0.7 0.7 0.0 1.0"/>
+      </material>
+    </visual>
+    <collision>
+      <!-- <origin xyz="0 0 ${wheel_radius + base_height/2.0}" rpy="0 0 0"/> -->
+      <origin xyz="-0.0055 0.0045 0" rpy="0 0 0"/>
+      <geometry>
+        <!-- <box size="${base_length} ${base_width} ${base_height}"/> -->
+        <mesh filename="file://${mesh_path}/myagv_base.dae" scale="1 1 1"/>
+      </geometry>
+      <surface>
+        <contact>
+          <ode/>
+        </contact>
+        <friction>
+          <ode mu="1.0" mu2="1.0"/>
+        </friction>
+      </surface>
+    </collision>
+    <collision>
+      <!-- <origin xyz="0 0 ${wheel_radius + base_height/2.0}" rpy="0 0 0"/> -->
+      <origin xyz="-0.0055 0.0045 0" rpy="0 0 0"/>
+      <geometry>
+        <!-- <box size="${base_length} ${base_width} ${base_height}"/> -->
+        <mesh filename="file://${mesh_path}/myagv_up.dae" scale="1 1 1"/>
       </geometry>
       <surface>
@@ -94,14 +121,14 @@
                                origin_rpy="0 0 0"/>
       <visual>
-        <origin xyz="0 0 0" rpy="0 1.5708 0"/>
+        <origin xyz="0 0 0" rpy="1.5708 0 0"/>
         <geometry>
           <cylinder radius="${wheel_radius}" length="${wheel_width}"/>
         </geometry>
-        <material name="${name}_black">
-          <color rgba="0.1 0.1 0.1 1.0"/>
+        <material name="${name}_dark_gray">
+          <color rgba="0.2 0.2 0.2 1.0"/>
         </material>
       </visual>
       <collision>
-        <origin xyz="0 0 0" rpy="0 1.5708 0"/>
+        <origin xyz="0 0 0" rpy="1.5708 0 0"/>
         <geometry>
           <cylinder radius="${wheel_radius}" length="${wheel_width}"/>

Commit message: fix: param adjustment

File: myagv_description/urdf/myagv_gazebo.urdf.xacro (robot description, xacro)
@@ -13,7 +13,7 @@
   <xacro:property name="wheel_offset_x" value="0.10555"/>
   <xacro:property name="wheel_offset_y" value="0.10525"/>
-  <xacro:property name="imu_height" value="${wheel_radius + base_height + 0.05}"/>
-  <xacro:property name="lidar_height" value="${wheel_radius + base_height + 0.08}"/>
-  <xacro:property name="camera_height" value="${wheel_radius + base_height + 0.15}"/>
+  <xacro:property name="imu_height" value="${base_height}"/>
+  <xacro:property name="lidar_height" value="${wheel_radius + base_height}"/>
+  <xacro:property name="camera_height" value="${base_height / 2}"/>
   <xacro:property name="mesh_path" value="$(find myagv_description)/meshes"/>
   <xacro:property name="ros2_control_config_path" value="$(arg ros2_control_config)"/>
@@ -80,8 +80,6 @@
     </visual>
     <collision>
-      <!-- <origin xyz="0 0 ${wheel_radius + base_height/2.0}" rpy="0 0 0"/> -->
-      <origin xyz="-0.0055 0.0045 0" rpy="0 0 0"/>
-      <geometry>
-        <!-- <box size="${base_length} ${base_width} ${base_height}"/> -->
+      <origin xyz="-0.0055 0.0045 0" rpy="0 0 0"/>
+      <geometry>
         <mesh filename="file://${mesh_path}/myagv_base.dae" scale="1 1 1"/>
       </geometry>
@@ -96,8 +94,6 @@
     </collision>
     <collision>
-      <!-- <origin xyz="0 0 ${wheel_radius + base_height/2.0}" rpy="0 0 0"/> -->
-      <origin xyz="-0.0055 0.0045 0" rpy="0 0 0"/>
-      <geometry>
-        <!-- <box size="${base_length} ${base_width} ${base_height}"/> -->
+      <origin xyz="-0.0055 0.0045 0" rpy="0 0 0"/>
+      <geometry>
         <mesh filename="file://${mesh_path}/myagv_up.dae" scale="1 1 1"/>
       </geometry>
@@ -178,5 +174,5 @@
     <inertial>
       <mass value="0.2"/>
-      <origin xyz="0 0 ${lidar_height}" rpy="0 0 0"/>
+      <origin xyz="0 0 0" rpy="0 0 0"/>
       <inertia ixx="2e-4" ixy="0" ixz="0" iyy="2e-4" iyz="0" izz="2e-4"/>
     </inertial>
@@ -184,5 +180,5 @@
       <origin xyz="0 0 0" rpy="0 0 0"/>
       <geometry>
-        <cylinder radius="0.04" length="0.05"/>
+        <cylinder radius="0.0285" length="0.025"/>
       </geometry>
       <material name="lidar_gray">
@@ -190,20 +186,14 @@
       </material>
     </visual>
-    <collision>
-      <origin xyz="0 0 0" rpy="0 0 0"/>
-      <geometry>
-        <cylinder radius="0.04" length="0.05"/>
-      </geometry>
-    </collision>
   </link>
   <joint name="lidar_joint" type="fixed">
     <parent link="base_link"/>
     <child link="lidar_link"/>
-    <origin xyz="0 0 ${lidar_height}" rpy="0 0 0"/>
+    <origin xyz="0.069 0 0.1" rpy="0 0 0"/>
   </joint>
   <link name="camera_link">
     <inertial>
       <mass value="0.2"/>
-      <origin xyz="0.05 0 ${camera_height}" rpy="0 0 0"/>
+      <origin xyz="0 0 0" rpy="0 0 0"/>
       <inertia ixx="1e-4" ixy="0" ixz="0" iyy="1e-4" iyz="0" izz="1e-4"/>
     </inertial>
@@ -211,5 +201,5 @@
       <origin xyz="0 0 0" rpy="0 0 0"/>
       <geometry>
-        <box size="0.08 0.04 0.04"/>
+        <box size="0.04 0.02 0.02"/>
       </geometry>
       <material name="camera_black">
@@ -217,15 +207,9 @@
       </material>
     </visual>
-    <collision>
-      <origin xyz="0 0 0" rpy="0 0 0"/>
-      <geometry>
-        <box size="0.08 0.04 0.04"/>
-      </geometry>
-    </collision>
   </link>
   <joint name="camera_joint" type="fixed">
     <parent link="base_link"/>
     <child link="camera_link"/>
-    <origin xyz="0.05 0 ${camera_height}" rpy="0 0 0"/>
+    <origin xyz="0.125 0 0.075" rpy="0 0 0"/>
   </joint>
   <!-- ros2_control hardware interface for wheels -->

Commit message: fix: sensor xyz param adjustment

File: myagv_description/urdf/myagv_gazebo.urdf.xacro (robot description, xacro)
@@ -159,32 +159,11 @@
                     xyz="${-wheel_offset_x} ${-wheel_offset_y} ${wheel_radius}"/>
   <!-- Sensor frames -->
-  <link name="imu_link">
-    <inertial>
-      <mass value="0.05"/>
-      <origin xyz="0 0 ${imu_height}" rpy="0 0 0"/>
-      <inertia ixx="1e-5" ixy="0" ixz="0" iyy="1e-5" iyz="0" izz="1e-5"/>
-    </inertial>
-  </link>
+  <link name="imu_link"/>
   <joint name="imu_joint" type="fixed">
     <parent link="base_link"/>
     <child link="imu_link"/>
-    <origin xyz="0 0 ${imu_height}" rpy="0 0 0"/>
-  </joint>
-  <link name="lidar_link">
-    <inertial>
-      <mass value="0.2"/>
-      <origin xyz="0 0 0" rpy="0 0 0"/>
-      <inertia ixx="2e-4" ixy="0" ixz="0" iyy="2e-4" iyz="0" izz="2e-4"/>
-    </inertial>
-    <visual>
-      <origin xyz="0 0 0" rpy="0 0 0"/>
-      <geometry>
-        <cylinder radius="0.0285" length="0.025"/>
-      </geometry>
-      <material name="lidar_gray">
-        <color rgba="0.3 0.3 0.3 1.0"/>
-      </material>
-    </visual>
-  </link>
+    <origin xyz="0 0 ${base_height / 2}" rpy="0 0 0"/>
+  </joint>
+  <link name="lidar_link"/>
   <joint name="lidar_joint" type="fixed">
     <parent link="base_link"/>
@@ -192,20 +171,5 @@
     <origin xyz="0.069 0 0.1" rpy="0 0 0"/>
   </joint>
-  <link name="camera_link">
-    <inertial>
-      <mass value="0.2"/>
-      <origin xyz="0 0 0" rpy="0 0 0"/>
-      <inertia ixx="1e-4" ixy="0" ixz="0" iyy="1e-4" iyz="0" izz="1e-4"/>
-    </inertial>
-    <visual>
-      <origin xyz="0 0 0" rpy="0 0 0"/>
-      <geometry>
-        <box size="0.04 0.02 0.02"/>
-      </geometry>
-      <material name="camera_black">
-        <color rgba="0.15 0.15 0.15 1.0"/>
-      </material>
-    </visual>
-  </link>
+  <link name="camera_link"/>
   <joint name="camera_joint" type="fixed">
     <parent link="base_link"/>

Commit message: feat: add sensor plugin

File: myagv_description/urdf/myagv_gazebo.urdf.xacro (robot description, xacro)
@@ -169,5 +169,5 @@
     <parent link="base_link"/>
     <child link="lidar_link"/>
-    <origin xyz="0.069 0 0.1" rpy="0 0 0"/>
+    <origin xyz="0.069 0 0.105" rpy="0 0 0"/>
   </joint>
   <link name="camera_link"/>
@@ -209,3 +209,85 @@
     </plugin>
   </gazebo>
+  <gazebo>
+    <plugin name="gazebo_ros_p3d" filename="libgazebo_ros_p3d.so">
+      <update_rate>50.0</update_rate>
+      <body_name>base_link</body_name>
+      <frame_name>odom</frame_name>
+      <child_frame_name>base_link</child_frame_name>
+      <publish_tf>true</publish_tf>
+      <gaussian_noise>0.0001</gaussian_noise>
+      <ros>
+        <remapping>~/odom:=/odom</remapping>
+      </ros>
+    </plugin>
+  </gazebo>
+  <gazebo reference="imu_link">
+    <sensor type="imu" name="myagv_imu">
+      <always_on>true</always_on>
+      <update_rate>50.0</update_rate>
+      <imu>
+        <topic>/imu/data</topic>
+        <gaussian_noise>0.0001</gaussian_noise>
+      </imu>
+      <plugin name="gazebo_ros_imu_sensor" filename="libgazebo_ros_imu_sensor.so">
+        <ros>
+          <remapping>~/out:=/imu</remapping>
+        </ros>
+      </plugin>
+    </sensor>
+  </gazebo>
+  <gazebo reference="lidar_link">
+    <sensor type="ray" name="myagv_lidar">
+      <always_on>true</always_on>
+      <pose>0 0 0 0 0 0</pose>
+      <update_rate>7.0</update_rate>
+      <visualize>true</visualize>
+      <ray>
+        <scan>
+          <horizontal>
+            <samples>432</samples>
+            <resolution>1</resolution>
+            <min_angle>-3.1415926535</min_angle>
+            <max_angle> 3.1415926535</max_angle>
+          </horizontal>
+        </scan>
+        <range>
+          <min>0.12</min>
+          <max>8.0</max>
+          <resolution>0.01</resolution>
+        </range>
+        <noise>
+          <type>gaussian</type>
+          <mean>0.0</mean>
+          <stddev>0.01</stddev>
+        </noise>
+      </ray>
+      <plugin name="gazebo_ros_ray_sensor" filename="libgazebo_ros_ray_sensor.so">
+        <output_type>sensor_msgs/LaserScan</output_type>
+        <frame_name>lidar_link</frame_name>
+        <ros>
+          <remapping>~/out:=/scan</remapping>
+        </ros>
+      </plugin>
+    </sensor>
+  </gazebo>
+  <gazebo reference="camera_link">
+    <sensor type="camera" name="myagv_camera">
+      <always_on>true</always_on>
+      <update_rate>30.0</update_rate>
+      <camera>
+        <horizontal_fov>1.047</horizontal_fov>
+        <image>
+          <width>640</width>
+          <height>480</height>
+          <format>R8G8B8</format>
+        </image>
+        <clip>
+          <near>0.1</near>
+          <far>100.0</far>
+        </clip>
+      </camera>
+      <plugin name="gazebo_ros_camera" filename="libgazebo_ros_camera.so"/>
+    </sensor>
+  </gazebo>
 </robot>

Commit message: fix: modify xacro sensor links

File: myagv_description/urdf/myagv_gazebo.urdf.xacro (robot description, xacro)
@@ -13,7 +13,4 @@
   <xacro:property name="wheel_offset_x" value="0.10555"/>
   <xacro:property name="wheel_offset_y" value="0.10525"/>
-  <xacro:property name="imu_height" value="${base_height}"/>
-  <xacro:property name="lidar_height" value="${wheel_radius + base_height}"/>
-  <xacro:property name="camera_height" value="${base_height / 2}"/>
   <xacro:property name="mesh_path" value="$(find myagv_description)/meshes"/>
   <xacro:property name="ros2_control_config_path" value="$(arg ros2_control_config)"/>
@@ -60,5 +57,5 @@
                         size_y="${base_width}"
                         size_z="${base_height}"
-                        origin_xyz="0 0 ${wheel_radius + base_height/2.0}"/>
+                        origin_xyz="0 0 0"/>
     <visual>
       <origin xyz="-0.0055 0.0045 0" rpy="0 0 0"/>
@@ -115,5 +112,5 @@
                                length="${wheel_width}"
                                origin_xyz="0 0 0"
-                               origin_rpy="0 0 0"/>
+                               origin_rpy="0 1.5708 0"/>
       <visual>
         <origin xyz="0 0 0" rpy="1.5708 0 0"/>
@@ -121,6 +118,6 @@
           <cylinder radius="${wheel_radius}" length="${wheel_width}"/>
         </geometry>
-        <material name="${name}_dark_gray">
-          <color rgba="0.2 0.2 0.2 1.0"/>
+        <material name="${name}_material">
+          <color rgba="0.3 0.3 0.3 1"/>
         </material>
       </visual>
@@ -135,5 +132,5 @@
           </contact>
           <friction>
-            <ode mu="1.2" mu2="1.2"/>
+            <ode mu="1.0" mu2="1.0"/>
           </friction>
         </surface>
@@ -141,44 +138,43 @@
     </link>
     <joint name="${name}_joint" type="continuous">
+      <origin xyz="${xyz}" rpy="0 0 0"/>
       <parent link="${parent}"/>
       <child link="${name}"/>
-      <origin xyz="${xyz}" rpy="0 0 0"/>
       <axis xyz="0 1 0"/>
-      <limit effort="20" velocity="25"/>
-      <dynamics damping="0.1" friction="0.05"/>
+      <dynamics friction="0.0" damping="0.0"/>
+      <limit upper="0" lower="0" effort="100.0" velocity="100.0"/>
     </joint>
   </xacro:macro>
   <!-- Wheels -->
-  <xacro:wheel_link name="front_left_wheel" parent="base_link"
-                    xyz="${wheel_offset_x} ${wheel_offset_y} ${wheel_radius}"/>
-  <xacro:wheel_link name="front_right_wheel" parent="base_link"
-                    xyz="${wheel_offset_x} ${-wheel_offset_y} ${wheel_radius}"/>
-  <xacro:wheel_link name="rear_left_wheel" parent="base_link"
-                    xyz="${-wheel_offset_x} ${wheel_offset_y} ${wheel_radius}"/>
-  <xacro:wheel_link name="rear_right_wheel" parent="base_link"
-                    xyz="${-wheel_offset_x} ${-wheel_offset_y} ${wheel_radius}"/>
-  <!-- Sensor frames -->
+  <xacro:wheel_link name="front_left_wheel" parent="base_link" xyz="${wheel_offset_x} ${wheel_offset_y} ${wheel_radius}"/>
+  <xacro:wheel_link name="front_right_wheel" parent="base_link" xyz="${wheel_offset_x} ${-wheel_offset_y} ${wheel_radius}"/>
+  <xacro:wheel_link name="rear_left_wheel" parent="base_link" xyz="${-wheel_offset_x} ${wheel_offset_y} ${wheel_radius}"/>
+  <xacro:wheel_link name="rear_right_wheel" parent="base_link" xyz="${-wheel_offset_x} ${-wheel_offset_y} ${wheel_radius}"/>
+  <!-- Base Link to IMU -->
   <link name="imu_link"/>
-  <joint name="imu_joint" type="fixed">
+  <joint name="base_imu_joint" type="fixed">
     <parent link="base_link"/>
     <child link="imu_link"/>
     <origin xyz="0 0 ${base_height / 2}" rpy="0 0 0"/>
   </joint>
+  <!-- Lidar -->
   <link name="lidar_link"/>
-  <joint name="lidar_joint" type="fixed">
+  <joint name="base_lidar_joint" type="fixed">
     <parent link="base_link"/>
     <child link="lidar_link"/>
-    <origin xyz="0.069 0 0.105" rpy="0 0 0"/>
-  </joint>
+    <origin xyz="0.065 0 0.105" rpy="0 0 0"/>
+  </joint>
+  <!-- Camera -->
   <link name="camera_link"/>
-  <joint name="camera_joint" type="fixed">
+  <joint name="base_camera_joint" type="fixed">
     <parent link="base_link"/>
     <child link="camera_link"/>
-    <origin xyz="0.125 0 0.075" rpy="0 0 0"/>
-  </joint>
-  <!-- ros2_control hardware interface for wheels -->
-  <ros2_control name="myagv_system" type="system">
+    <origin xyz="0.14 0 0.07225" rpy="0 0 0"/>
+  </joint>
+  <!-- ros2_control block -->
+  <ros2_control name="myagv_base" type="system">
     <hardware>
       <plugin>gazebo_ros2_control/GazeboSystem</plugin>
+      <param name="robot_description">myagv</param>
     </hardware>
     <joint name="front_left_wheel_joint">

Commit message: fix: modify params

File: myagv_description/urdf/myagv_gazebo.urdf.xacro (robot description, xacro)
@@ -8,4 +8,5 @@
   <xacro:property name="base_height" value="0.11"/>
   <xacro:property name="base_mass" value="4.16"/>
+  <xacro:property name="base_mesh_xyz" value="-0.0055 0.00448 0"/>
   <xacro:property name="wheel_radius" value="0.04"/>
   <xacro:property name="wheel_width" value="0.032"/>
@@ -59,5 +60,5 @@
                         origin_xyz="0 0 0"/>
     <visual>
-      <origin xyz="-0.0055 0.0045 0" rpy="0 0 0"/>
+      <origin xyz="${base_mesh_xyz}" rpy="0 0 0"/>
       <geometry>
         <mesh filename="file://${mesh_path}/myagv_base.dae" scale="1 1 1"/>
@@ -68,5 +69,5 @@
     </visual>
     <visual>
-      <origin xyz="-0.0055 0.0045 0" rpy="0 0 0"/>
+      <origin xyz="${base_mesh_xyz}" rpy="0 0 0"/>
       <geometry>
         <mesh filename="file://${mesh_path}/myagv_up.dae" scale="1 1 1"/>
@@ -77,5 +78,5 @@
     </visual>
     <collision>
-      <origin xyz="-0.0055 0.0045 0" rpy="0 0 0"/>
+      <origin xyz="${base_mesh_xyz}" rpy="0 0 0"/>
       <geometry>
         <mesh filename="file://${mesh_path}/myagv_base.dae" scale="1 1 1"/>
@@ -91,5 +92,5 @@
     </collision>
     <collision>
-      <origin xyz="-0.0055 0.0045 0" rpy="0 0 0"/>
+      <origin xyz="${base_mesh_xyz}" rpy="0 0 0"/>
       <geometry>
         <mesh filename="file://${mesh_path}/myagv_up.dae" scale="1 1 1"/>
@@ -176,5 +177,4 @@
     <hardware>
       <plugin>gazebo_ros2_control/GazeboSystem</plugin>
-      <param name="robot_description">myagv</param>
     </hardware>
     <joint name="front_left_wheel_joint">
@@ -205,17 +205,4 @@
     </plugin>
   </gazebo>
-  <gazebo>
-    <plugin name="gazebo_ros_p3d" filename="libgazebo_ros_p3d.so">
-      <update_rate>50.0</update_rate>
-      <body_name>base_link</body_name>
-      <frame_name>odom</frame_name>
-      <child_frame_name>base_link</child_frame_name>
-      <publish_tf>true</publish_tf>
-      <gaussian_noise>0.0001</gaussian_noise>
-      <ros>
-        <remapping>~/odom:=/odom</remapping>
-      </ros>
-    </plugin>
-  </gazebo>
   <gazebo reference="imu_link">
     <sensor type="imu" name="myagv_imu">
@@ -223,5 +210,4 @@
       <update_rate>50.0</update_rate>
       <imu>
-        <topic>/imu/data</topic>
         <gaussian_noise>0.0001</gaussian_noise>
       </imu>
@@ -244,6 +230,8 @@
             <samples>432</samples>
             <resolution>1</resolution>
-            <min_angle>-3.1415926535</min_angle>
-            <max_angle> 3.1415926535</max_angle>
+            <!-- <min_angle>-3.1415926535</min_angle>
+            <max_angle> 3.1415926535</max_angle> -->
+            <min_angle>-2.2689280082</min_angle>
+            <max_angle> 2.2689280082</max_angle>
           </horizontal>
         </scan>
