Commit message: fix: inertial for cylinder

File: myagv_description/urdf/myagv_gazebo.urdf.xacro (robot description, xacro)
@@ -22,9 +22,6 @@
       <origin xyz="${origin_xyz}" rpy="0 0 0"/>
       <inertia
-        ixx="${mass/12.0 * (size_y*size_y + size_z*size_z)}"
-        ixy="0.0"
-        ixz="0.0"
-        iyy="${mass/12.0 * (size_x*size_x + size_z*size_z)}"
-        iyz="0.0"
+        ixx="${mass/12.0 * (size_y*size_y + size_z*size_z)}" ixy="0.0" ixz="0.0"
+        iyy="${mass/12.0 * (size_x*size_x + size_z*size_z)}" iyz="0.0"
         izz="${mass/12.0 * (size_x*size_x + size_y*size_y)}"/>
     </inertial>
@@ -35,10 +32,7 @@
       <origin xyz="${origin_xyz}" rpy="${origin_rpy}"/>
       <inertia
-        ixx="${mass/12.0 * (3*radius*radius + length*length)}"
-        ixy="0.0"
-        ixz="0.0"
-        iyy="${mass/2.0 * radius*radius}"
-        iyz="0.0"
-        izz="${mass/12.0 * (3*radius*radius + length*length)}"/>
+        ixx="${mass/12.0 * (3*radius*radius + length*length)}" ixy="0.0" ixz="0.0"
+        iyy="${mass/12.0 * (3*radius*radius + length*length)}" iyz="0.0"
+        izz="${mass/2.0 * radius*radius}"/>
     </inertial>
   </xacro:macro>
@@ -48,6 +42,5 @@
     <parent link="base_footprint"/>
     <child link="base_link"/>
-    <!-- <origin xyz="0 0.0045 0" rpy="0 0 0"/> -->
-    <origin xyz="0 0 0" rpy="0 0 0"/>
+    <origin xyz="0 0 ${wheel_radius}" rpy="0 0 0"/>
     <axis xyz="0 0 1"/>
   </joint>
@@ -82,12 +75,4 @@
         <mesh filename="file://${mesh_path}/myagv_base.dae" scale="1 1 1"/>
       </geometry>
-      <surface>
-        <contact>
-          <ode/>
-        </contact>
-        <friction>
-          <ode mu="1.0" mu2="1.0"/>
-        </friction>
-      </surface>
     </collision>
     <collision>
@@ -96,12 +81,4 @@
         <mesh filename="file://${mesh_path}/myagv_up.dae" scale="1 1 1"/>
       </geometry>
-      <surface>
-        <contact>
-          <ode/>
-        </contact>
-        <friction>
-          <ode mu="1.0" mu2="1.0"/>
-        </friction>
-      </surface>
     </collision>
   </link>
@@ -113,5 +90,5 @@
                                length="${wheel_width}"
                                origin_xyz="0 0 0"
-                               origin_rpy="0 1.5708 0"/>
+                               origin_rpy="1.5708 0 0"/>
       <visual>
         <origin xyz="0 0 0" rpy="1.5708 0 0"/>
@@ -128,12 +105,4 @@
           <cylinder radius="${wheel_radius}" length="${wheel_width}"/>
         </geometry>
-        <surface>
-          <contact>
-            <ode/>
-          </contact>
-          <friction>
-            <ode mu="1.0" mu2="1.0"/>
-          </friction>
-        </surface>
       </collision>
     </link>
@@ -143,6 +112,6 @@
       <child link="${name}"/>
       <axis xyz="0 1 0"/>
-      <dynamics friction="0.0" damping="0.0"/>
-      <limit upper="0" lower="0" effort="100.0" velocity="100.0"/>
+      <!-- <dynamics friction="0.0" damping="0.0"/>
+      <limit upper="0" lower="0" effort="100.0" velocity="100.0"/> -->
     </joint>
   </xacro:macro>
