Commit message: feat: integrate slam, nav2 with gzb

File: myagv_description/urdf/myagv_gazebo_skid.urdf.xacro (robot description, xacro)
@@ -3,10 +3,9 @@
   <!-- Arguments -->
   <xacro:arg name="ros2_control_config" default=""/>
-  <!-- Dimensions (approximate, tune with measured data when available) -->
+  <!-- Dimensions -->
   <xacro:property name="base_length" value="0.31115"/>
   <xacro:property name="base_width" value="0.23"/>
   <xacro:property name="base_height" value="0.11"/>
   <xacro:property name="base_mass" value="4.16"/>
-  <xacro:property name="base_mesh_xyz" value="-0.0055 0.00448 0"/>
   <xacro:property name="wheel_radius" value="0.04"/>
   <xacro:property name="wheel_width" value="0.032"/>
@@ -15,5 +14,5 @@
   <xacro:property name="wheel_offset_y" value="0.10525"/>
   <xacro:property name="mesh_path" value="$(find myagv_description)/meshes"/>
-  <xacro:property name="ros2_control_config_path" value="$(arg ros2_control_config)"/>
+  <xacro:property name="base_mesh_xyz" value="-0.0055 0.00448 0"/>
   <!-- Helper macros -->
   <xacro:macro name="box_inertial" params="mass size_x size_y size_z origin_xyz">
@@ -22,6 +21,9 @@
       <origin xyz="${origin_xyz}" rpy="0 0 0"/>
       <inertia
-        ixx="${mass/12.0 * (size_y*size_y + size_z*size_z)}" ixy="0.0" ixz="0.0"
-        iyy="${mass/12.0 * (size_x*size_x + size_z*size_z)}" iyz="0.0"
+        ixx="${mass/12.0 * (size_y*size_y + size_z*size_z)}"
+        ixy="0.0"
+        ixz="0.0"
+        iyy="${mass/12.0 * (size_x*size_x + size_z*size_z)}"
+        iyz="0.0"
         izz="${mass/12.0 * (size_x*size_x + size_y*size_y)}"/>
     </inertial>
@@ -32,6 +34,9 @@
       <origin xyz="${origin_xyz}" rpy="${origin_rpy}"/>
       <inertia
-        ixx="${mass/12.0 * (3*radius*radius + length*length)}" ixy="0.0" ixz="0.0"
-        iyy="${mass/12.0 * (3*radius*radius + length*length)}" iyz="0.0"
+        ixx="${mass/12.0 * (3*radius*radius + length*length)}"
+        ixy="0.0"
+        ixz="0.0"
+        iyy="${mass/12.0 * (3*radius*radius + length*length)}"
+        iyz="0.0"
         izz="${mass/2.0 * radius*radius}"/>
     </inertial>
@@ -45,5 +50,5 @@
     <axis xyz="0 0 1"/>
   </joint>
-  <!-- Base link with visuals and collision -->
+  <!-- Base link -->
   <link name="base_link">
     <xacro:box_inertial mass="${base_mass}"
@@ -58,5 +63,5 @@
       </geometry>
       <material name="black">
-          <color rgba="0.7 0.7 0.0 1.0"/>
+        <color rgba="0.7 0.7 0.0 1.0"/>
       </material>
     </visual>
@@ -67,5 +72,5 @@
       </geometry>
       <material name="black">
-          <color rgba="0.7 0.7 0.0 1.0"/>
+        <color rgba="0.7 0.7 0.0 1.0"/>
       </material>
     </visual>
@@ -105,4 +110,13 @@
           <cylinder radius="${wheel_radius}" length="${wheel_width}"/>
         </geometry>
+        <surface>
+          <contact>
+            <ode kp="5e4" kd="5.0" soft_cfm="1e-6" soft_erp="0.8"/>
+          </contact>
+          <friction>
+            <ode mu="0.6" mu2="0.01" slip1="0.0" slip2="2.0"/>
+            <fdir1>1 0 0</fdir1>
+          </friction>
+        </surface>
       </collision>
     </link>
@@ -119,12 +133,11 @@
   <xacro:wheel_link name="rear_left_wheel" parent="base_link" xyz="${-wheel_offset_x} ${wheel_offset_y} ${wheel_radius}"/>
   <xacro:wheel_link name="rear_right_wheel" parent="base_link" xyz="${-wheel_offset_x} ${-wheel_offset_y} ${wheel_radius}"/>
-  <!-- Base Link to IMU -->
+  <!-- Sensors and auxiliary links -->
   <link name="imu_link"/>
   <joint name="base_imu_joint" type="fixed">
     <parent link="base_link"/>
     <child link="imu_link"/>
-    <origin xyz="0 0 ${base_height / 2}" rpy="0 0 0"/>
-  </joint>
-  <!-- Lidar -->
+    <origin xyz="0 0 ${base_height/2}" rpy="0 0 0"/>
+  </joint>
   <link name="lidar_link"/>
   <joint name="base_lidar_joint" type="fixed">
@@ -133,5 +146,4 @@
     <origin xyz="0.065 0 0.105" rpy="0 0 0"/>
   </joint>
-  <!-- Camera -->
   <link name="camera_link"/>
   <joint name="base_camera_joint" type="fixed">
@@ -140,34 +152,24 @@
     <origin xyz="0.14 0 0.07225" rpy="0 0 0"/>
   </joint>
-  <!-- ros2_control block -->
-  <ros2_control name="myagv_base" type="system">
-    <hardware>
-      <plugin>gazebo_ros2_control/GazeboSystem</plugin>
-    </hardware>
-    <joint name="front_left_wheel_joint">
-      <command_interface name="velocity"/>
-      <state_interface name="position"/>
-      <state_interface name="velocity"/>
-    </joint>
-    <joint name="front_right_wheel_joint">
-      <command_interface name="velocity"/>
-      <state_interface name="position"/>
-      <state_interface name="velocity"/>
-    </joint>
-    <joint name="rear_left_wheel_joint">
-      <command_interface name="velocity"/>
-      <state_interface name="position"/>
-      <state_interface name="velocity"/>
-    </joint>
-    <joint name="rear_right_wheel_joint">
-      <command_interface name="velocity"/>
-      <state_interface name="position"/>
-      <state_interface name="velocity"/>
-    </joint>
-  </ros2_control>
-  <!-- Gazebo ros2_control plugin -->
+  <!-- Gazebo skid-steer plugin -->
   <gazebo>
-    <plugin name="gazebo_ros2_control" filename="libgazebo_ros2_control.so">
-      <parameters>${ros2_control_config_path}</parameters>
+    <plugin name="skid_steer_drive" filename="libgazebo_ros_skid_steer_drive.so">
+      <ros>
+        <remapping>cmd_vel:=/cmd_vel</remapping>
+        <remapping>odom:=/odom</remapping>
+      </ros>
+      <left_front_joint>front_left_wheel_joint</left_front_joint>
+      <left_rear_joint>rear_left_wheel_joint</left_rear_joint>
+      <right_front_joint>front_right_wheel_joint</right_front_joint>
+      <right_rear_joint>rear_right_wheel_joint</right_rear_joint>
+      <wheel_separation>${2 * wheel_offset_y}</wheel_separation>
+      <wheel_diameter>${2 * wheel_radius}</wheel_diameter>
+      <max_wheel_torque>15.0</max_wheel_torque>
+      <max_wheel_acceleration>5.0</max_wheel_acceleration>
+      <publish_odom>true</publish_odom>
+      <publish_tf>false</publish_tf>
+      <odometry_frame>odom</odometry_frame>
+      <robot_base_frame>base_footprint</robot_base_frame>
+      <update_rate>50.0</update_rate>
     </plugin>
   </gazebo>
@@ -197,6 +199,4 @@
             <samples>432</samples>
             <resolution>1</resolution>
-            <!-- <min_angle>-3.1415926535</min_angle>
-            <max_angle> 3.1415926535</max_angle> -->
             <min_angle>-2.2689280082</min_angle>
             <max_angle> 2.2689280082</max_angle>
